File: KiCAD/HealthBand/PPG.sch (KiCad schematic (older format))
At the start: 0 parts

Commit message: Need more work on component selection
Parts:
- added U?: MAX30101EFD+T, custom_footprints:MAX30101EFD&plus_T, symbol MAX30101EFDT:MAX30101EFD+T
Changed lines of the file:
@@
 Comment4 ""
 $EndDescr
+$Comp
+L MAX30101EFDT:MAX30101EFD+T U?
+U 1 1 601D47FD
+P 4630 2990
+F 0 "U?" H 5430 3477 60  0000 C CNN
+F 1 "MAX30101EFD+T" H 5430 3371 60  0000 C CNN
+F 2 "custom_footprints:MAX30101EFD&plus_T" H 5430 3330 60  0001 C CNN
+F 3 "" H 4630 2990 60  0000 C CNN
+	1    4630 2990
+	1    0    0    -1
+$EndComp
 $EndSCHEMATC
